File: keyBoard.sch (EAGLE design)
At the start: 34 parts, among them IC1 317EMP, J3 USB_A_PTH_MALE, J4 ISCP, U1 MCP73833-FCI/UN, Y2 16MHz

Commit message: updating board
Parts:
- added C7, C9: 1.0uF, SparkFun-Capacitors:1.0UF-0603-16V-10%
- added C8: 10uF, SparkFun-Capacitors:10UF-0603-6.3V-20%
- added D4: Yellow, SparkFun-LED:LED-YELLOW0603
- added R10, R11, R15, R9: 10k, SparkFun-Resistors:10KOHM-0603-1/10W-1%
- added R14: 1k, SparkFun-Resistors:1KOHM-0603-1/10W-1%
- added R_D+, R_D-: 22, SparkFun-Resistors:22OHM-0603-1/10W-1%
- added S1: (no value), SparkFun-Switches:JOYSTICK_MINI
- added U2: MCP73831, SparkFun-IC-Power:MCP73831
- R7, R8: value 22 -> 10k; device SparkFun-Resistors:22OHM-0603-1/10W-1% -> SparkFun-Resistors:10KOHM-0603-1/10W-1%
- U1: value MCP73833-FCI/UN -> MCP73833
Connections:
- new net CTR: R11.1, S1.CENT, U$1.PD6(T1/ADC9/!OC4D)
- new net DOWN: R10.1, S1.DOWN
- new net N$5: D4.C, R14.2
- new net N$6: R15.2, U2.PROG
- new net STAT: R14.1, U2.STAT
- new net UCAP: C7.1, U$1.UCAP
- new net UP: R9.1, S1.UP, U$1.PD7(OC4D/ADC10/T0)
- net +3V3: now also C9.1, R10.2, R11.2, R7.2, R8.2, R9.2; no longer U$1.UCAP
- net D+: now also R_D+.2; no longer R7.2
- net D-: now also R_D-.2; no longer R8.2
- net GND: now also C7.2, C8.2, C9.2, R15.1, S1.GND, U2.VSS
- net N$2: now also R_D+.1; no longer R7.1
- net N$3: now also R_D-.1; no longer R8.1
- net SCL: now also R7.1
- net SDA: now also R8.1
- net VBAT: now also C8.1, U2.VBAT
- net VBUS: now also D4.A, U$1.UVCC, U2.VIN
Other:
- moved on the sheet: C6, JP1, R7, R8

Commit message: editted gitignore & deleted some files
Parts:
- removed C1: 10uF, SparkFun-Capacitors:10UF-0603-6.3V-20%
- removed D2: Yellow, SparkFun-LED:LED-YELLOW0603
- removed D3: RED, SparkFun-LED:LED-RED0603
- removed R1, R2, R3: 1k, SparkFun-Resistors:1KOHM-0603-1/10W-1%
- removed R4: 2.0k, SparkFun-Resistors:2.0KOHM-0603-1/10W-5%
- removed R5: 10k, SparkFun-Resistors:10KOHM-0603-1/10W-1%
- removed U1: MCP73833, Microchip-MCP73833-FCI_UN:MCP73833-FCI/UN
- D1: value GREEN -> MBR120; device SparkFun-LED:LED-GREEN0603 -> adafruit:DIODE_SOD-123FL
- J2: value (none) -> FINGER_SCAN
- JP1: value (none) -> SCREEN
- S1: value (none) -> JOYSTICK
- U3: value (none) -> nRF51
Connections:
- removed net N$1: D2.C, R2.2
- removed net N$4: D1.C, R1.2
- removed net N$7: D3.C, R3.2
- removed net PG: R3.1, U1.*PG
- removed net PROG: R4.2, U1.PROG
- removed net STAT1: R2.1, U1.STAT1
- removed net STAT2: R1.1, U1.STAT2
- removed net THERM: R5.2, U1.THERM
- net GND: no longer C1.2, R4.1, R5.1, U1.VSS
- net VBAT: now also D1.A; no longer C1.1, IC1.VI, U1.VBAT, U1.VBAT_2
- net VBUS: now also D1.C, IC1.VI; no longer D1.A, D2.A, D3.A, U1.VDD, U1.VDD_2
Other:
- moved on the sheet: C2, C8, D4, J2, J3, J4, JP1, R10, R11, R14, R15, R6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

Commit message: forgot to connect DOWN on the joystick
Connections:
- net DOWN: now also U$1.PD5(XCK/CTS)
Changed lines of the file:
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@@
 <setting verticaltext="up"/>
 </settings>
-<grid distance="25" unitdist="mil" unit="mil" style="lines" multiple="1" display="no" altdistance="0.01" altunitdist="inch" altunit="inch"/>
+<grid distance="0.1" unitdist="inch" unit="inch" style="lines" multiple="1" display="no" altdistance="0.01" altunitdist="inch" altunit="inch"/>
 <layers>
 <layer number="1" name="Top" color="4" fill="1" visible="no" active="no"/>
@@
 <label x="-114.3" y="-52.07" size="1.778" layer="95"/>
 </segment>
-</net>
+<segment>
+<pinref part="U$1" gate="G$1" pin="PD5(XCK/CTS)"/>
+<wire x1="226.06" y1="-93.98" x2="233.68" y2="-93.98" width="0.1524" layer="91"/>
+</segment>
+</net>

Commit message: final board, mid-semester arduino proof of concept, non-working disjoint AVR C code
Parts:
- removed D4: Yellow, SparkFun-LED:LED-YELLOW0603
- removed Y2: 16MHz, SparkFun-Clocks:CRYSTAL-16MHZSMD-5X3.2
- added CHARGE: Yellow, SparkFun-LED:LED-YELLOW0603
- added Y1: 8MHz, SparkFun-Clocks:CRYSTAL-8MHZSMD-5X3.2
Connections:
- removed net CONNECTED: CONN.A, U3.P0.19
- removed net N$10: MODE.C, R12.2
- removed net N$13: CONN.C, R13.2
- removed net N$5: D4.C, R14.2
- new net CONNECTION: R13.2, U3.P0.19
- new net N$1: CHARGE.A, R14.2
- new net N$4: MODE.A, R12.1
- new net N$7: CONN.A, R13.1
- net GND: now also CONN.C, MODE.C; no longer R12.1, R13.1
- net MODE: now also R12.2; no longer MODE.A
- net STAT: now also CHARGE.C; no longer R14.1
- net VBUS: now also R14.1; no longer D4.A
- net XTAL1: now also Y1.2; no longer Y2.2
- net XTAL2: now also Y1.1; no longer Y2.1
Other:
- moved on the sheet: CONN, MODE, R12, R13, R14
